Commit message: 修复仿真中夹爪角度错误的bug

File: src/robot_arm/urdf/robot_arm.urdf (robot description, URDF)
Before this commit: robot robot_arm, 12 links, 11 joints
Joints:
- joint joint11_right: origin xyz=0.018 0.058 0.00565 rpy=3.1416 -1.5708 0 -> xyz=0.018 0.058 0.00565 rpy=0 -1.5708 0
- joint joint5: limit lower=-2.09 upper=2.09 effort=1.96 velocity=3.14 -> lower=-1.57 upper=1.57 effort=1.96 velocity=3.14
- joint joint6_left: limit lower=-0.628 upper=6.28 effort=1.96 velocity=3.14 -> lower=-0.2 upper=1.0 effort=1.96 velocity=3.14
- joint joint9_right: origin xyz=0.018 0.038 -0.00235 rpy=3.1416 -1.5708 0 -> xyz=0.018 0.038 -0.00235 rpy=0 -1.5708 0

Commit message: 为机械臂添加gazebo仿真控制器，修复了mimic随动关节的bug

File: src/robot_arm/urdf/robot_arm.urdf (robot description, URDF)
Before this commit: robot robot_arm, 12 links, 11 joints
Links:
- added link grasping_frame
- added link world
Joints:
- added joint fixed_base_joint: type fixed, parent world, child base_link
- added joint grasping_frame_joint: type fixed, parent link5, child grasping_frame, origin xyz=0.02248 0.12258 0.00595 rpy=1.5708 0 1.5708
