Commit message: 创建main_simulationlaunch文件，使棋盘和机械臂在同一个世界中

File: src/board_new/urdf/board_new.urdf (robot description, URDF)
Before this commit: robot board_new, 34 links, 33 joints
Joints:
- removed joint world_to_base
- added joint fixed_to_world: type fixed, parent world, child base_link, origin xyz=0 0 0.02 rpy=1.5708 0 0

File: src/robot_arm/urdf/robot_arm.xacro (robot description, xacro)
@@ -772,5 +772,5 @@
   <gazebo>
     <plugin name="gazebo_ros_control" filename="libgazebo_ros_control.so">
-      <robotNamespace>/robot_arm</robotNamespace>
+      <!-- <robotNamespace>/robot_arm</robotNamespace> -->
       <robotSimType>gazebo_ros_control/DefaultRobotHWSim</robotSimType>
     </plugin>
